File: circuit/smd.sch (EAGLE design)
At the start: 16 parts, among them IC1 AT90S2313S, Q1 16MHz, X1 USB-1X-2S-PLUG-A-THT

Commit message: smd layout: add status LEDs, cause status LEDs are always good \o/
Parts:
- added LED1, LED2: (no value), led:LEDSML0805
- added R7: (no value), rcl:R-EU_R0805
Connections:
- new net LED1: IC1.(TXD)PD1, LED1.C, LED2.A
- new net LED2: IC1.(RXD)PD0, R7.1
- new net N$2: LED1.A, LED2.C, R7.2
Other:
- note added: "Status LED"
Changed lines of the file:
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@@
 <part name="FRAME1" library="frames" deviceset="A5L-LOC" device="" value="vusb-i2c"/>
 <part name="X1" library="_con-usb_1" deviceset="USB-1X-2S" device="-PLUG-A-THT" value="USB-1X-2S-PLUG-A-THT"/>
+<part name="LED1" library="led" deviceset="LED" device="SML0805"/>
+<part name="LED2" library="led" deviceset="LED" device="SML0805"/>
+<part name="R7" library="rcl" deviceset="R-EU_" device="R0805"/>
 </parts>
 <sheets>
@@
 <wire x1="85.09" y1="53.34" x2="85.09" y2="4.064" width="0.1524" layer="97" style="longdash"/>
 <wire x1="86.36" y1="53.34" x2="116.84" y2="53.34" width="0.1524" layer="97" style="longdash"/>
-<wire x1="116.84" y1="53.34" x2="116.84" y2="129.54" width="0.1524" layer="97" style="longdash"/>
+<wire x1="116.84" y1="53.34" x2="116.84" y2="104.14" width="0.1524" layer="97" style="longdash"/>
+<wire x1="116.84" y1="104.14" x2="116.84" y2="129.54" width="0.1524" layer="97" style="longdash"/>
 <wire x1="116.84" y1="53.34" x2="180.34" y2="53.34" width="0.1524" layer="97" style="longdash"/>
 <text x="63.5" y="50.8" size="1.778" layer="97">USB Interface</text>
@@
 <text x="119.38" y="55.88" size="1.778" layer="97">I2C Interface</text>
 <text x="86.36" y="50.8" size="1.778" layer="97">SPI Interface</text>
+<wire x1="116.84" y1="104.14" x2="180.34" y2="104.14" width="0.1524" layer="97" style="longdash"/>
+<text x="119.38" y="106.68" size="1.778" layer="97">Status LED</text>
 </plain>
 <instances>
@@
 <instance part="FRAME1" gate="G$1" x="0" y="0"/>
 <instance part="X1" gate="G$1" x="17.78" y="30.48"/>
+<instance part="LED1" gate="G$1" x="152.4" y="121.92" rot="R90"/>
+<instance part="LED2" gate="G$1" x="154.94" y="114.3" rot="R270"/>
+<instance part="R7" gate="G$1" x="139.7" y="119.38"/>
 </instances>
 <busses>
@@
 </segment>
 </net>
+<net name="LED2" class="0">
+<segment>
+<pinref part="IC1" gate="G$1" pin="(RXD)PD0"/>
+<wire x1="76.2" y1="58.42" x2="78.74" y2="58.42" width="0.1524" layer="91"/>
+<wire x1="78.74" y1="58.42" x2="78.74" y2="55.88" width="0.1524" layer="91"/>
+<wire x1="101.6" y1="55.88" x2="78.74" y2="55.88" width="0.1524" layer="91"/>
+<label x="93.98" y="55.88" size="1.778" layer="95"/>
+</segment>
+<segment>
+<pinref part="R7" gate="G$1" pin="1"/>
+<wire x1="134.62" y1="119.38" x2="121.92" y2="119.38" width="0.1524" layer="91"/>
+<label x="124.46" y="119.38" size="1.778" layer="95"/>
+</segment>
+</net>
+<net name="LED1" class="0">
+<segment>
+<pinref part="IC1" gate="G$1" pin="(TXD)PD1"/>
+<wire x1="76.2" y1="60.96" x2="81.28" y2="60.96" width="0.1524" layer="91"/>
+<wire x1="81.28" y1="60.96" x2="81.28" y2="58.42" width="0.1524" layer="91"/>
+<wire x1="81.28" y1="58.42" x2="101.6" y2="58.42" width="0.1524" layer="91"/>
+<label x="93.98" y="58.42" size="1.778" layer="95"/>
+</segment>
+<segment>
+<pinref part="LED1" gate="G$1" pin="C"/>
+<wire x1="157.48" y1="121.92" x2="160.02" y2="121.92" width="0.1524" layer="91"/>
+<wire x1="160.02" y1="121.92" x2="160.02" y2="119.38" width="0.1524" layer="91"/>
+<pinref part="LED2" gate="G$1" pin="A"/>
+<wire x1="160.02" y1="119.38" x2="160.02" y2="114.3" width="0.1524" layer="91"/>
+<wire x1="160.02" y1="114.3" x2="157.48" y2="114.3" width="0.1524" layer="91"/>
+<wire x1="160.02" y1="119.38" x2="172.72" y2="119.38" width="0.1524" layer="91"/>
+<junction x="160.02" y="119.38"/>
+<label x="165.1" y="119.38" size="1.778" layer="95"/>
+</segment>
+</net>
+<net name="N$2" class="0">
+<segment>
+<pinref part="R7" gate="G$1" pin="2"/>
+<wire x1="144.78" y1="119.38" x2="147.32" y2="119.38" width="0.1524" layer="91"/>
+<wire x1="147.32" y1="119.38" x2="147.32" y2="121.92" width="0.1524" layer="91"/>
+<pinref part="LED1" gate="G$1" pin="A"/>
+<wire x1="147.32" y1="121.92" x2="149.86" y2="121.92" width="0.1524" layer="91"/>
+<wire x1="147.32" y1="119.38" x2="147.32" y2="114.3" width="0.1524" layer="91"/>
+<pinref part="LED2" gate="G$1" pin="C"/>
+<wire x1="147.32" y1="114.3" x2="149.86" y2="114.3" width="0.1524" layer="91"/>
+<junction x="147.32" y="119.38"/>
+</segment>
+</net>

Commit message: smd rev 1 at board house
Parts:
- LED1: value (none) -> act
- LED2: value (none) -> pwr
- R7: value (none) -> 150..1K
Changed lines of the file:
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@@
 <part name="FRAME1" library="frames" deviceset="A5L-LOC" device="" value="vusb-i2c"/>
 <part name="X1" library="_con-usb_1" deviceset="USB-1X-2S" device="-PLUG-A-THT" value="USB-1X-2S-PLUG-A-THT"/>
-<part name="LED1" library="led" deviceset="LED" device="SML0805"/>
-<part name="LED2" library="led" deviceset="LED" device="SML0805"/>
-<part name="R7" library="rcl" deviceset="R-EU_" device="R0805"/>
+<part name="LED1" library="led" deviceset="LED" device="SML0805" value="act"/>
+<part name="LED2" library="led" deviceset="LED" device="SML0805" value="pwr"/>
+<part name="R7" library="rcl" deviceset="R-EU_" device="R0805" value="150..1K"/>
 </parts>
 <sheets>
