File: circuit/circuit.brd (EAGLE design)
At the start: 41.6 x 34.3 mm, 16 parts, among them IC1 AT90S2313P, Q1 16MHz

Commit message: more baord layout improvements
Parts:
- moved JP2 15.2 mm to (36.8, 22.9)
- moved C4 11.4 mm to (36.8, 15.2)
- moved C5 11.4 mm to (36.8, 5.08)
- moved Q1 11.4 mm to (36.8, 10.2)
- moved JP1 1.27 mm to (3.81, 22.9)
Routing:
- net SDA: track 37.4 -> 46.4 mm
- net N$38: track 8.43 -> 11.3 mm
- net SCL: track 44.9 -> 47.2 mm, vias 0 -> 1
- net VCC: track 76.9 -> 78.0 mm
- net D+: track 14.1 -> 13.5 mm
- net D-: track 15.0 -> 14.5 mm
Other:
- board text added: "5V"
- board text added: "D+"
- board text added: "D-"
- board text added: "GND"
- board text added: "SCL"
- board text added: "SDA"
- board text added: "derf"
- board text added: "rev 1"
- board text added: "vusb-i2c"
- board text removed: "derf / vusb-i2c / rev 1"

Commit message: such layout, wow
Connections:
- net GND: now also JP2.1; no longer JP2.2
- net SCL: now also JP2.2; no longer JP2.1
- net SDA: now also JP2.3; no longer JP2.4
- net VCC: now also JP2.4; no longer JP2.3
Routing:
- net SDA: track 46.4 -> 43.1 mm
- net VCC: track 78.0 -> 79.6 mm
Changed lines of the file:
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@@
 <text x="5.715" y="23.495" size="1.016" layer="25">D-</text>
 <text x="5.715" y="20.955" size="1.016" layer="25">D+</text>
-<text x="38.735" y="26.035" size="1.016" layer="25">SDA</text>
-<text x="38.735" y="18.415" size="1.016" layer="25">SCL</text>
-<text x="38.735" y="23.495" size="1.016" layer="25">5V</text>
-<text x="38.735" y="20.955" size="1.016" layer="25">GND</text>
+<text x="38.735" y="23.495" size="1.016" layer="25">SDA</text>
+<text x="38.735" y="20.955" size="1.016" layer="25">SCL</text>
+<text x="38.735" y="26.035" size="1.016" layer="25">5V</text>
+<text x="38.735" y="18.415" size="1.016" layer="25">GND</text>
 </plain>
 <attributes>
@@
 <contactref element="JP1" pad="1"/>
 <contactref element="SV2" pad="6"/>
-<contactref element="JP2" pad="2"/>
 <polygon width="0.4064" layer="1" isolate="0.3048">
 <vertex x="0" y="34.29"/>
@@
 <vertex x="0" y="0"/>
 </polygon>
+<contactref element="JP2" pad="1"/>
 </signal>
 <signal name="N$37">
@@
 <contactref element="JP1" pad="4"/>
 <contactref element="SV2" pad="2"/>
-<contactref element="JP2" pad="3"/>
 <wire x1="27.94" y1="19.05" x2="27.94" y2="10.16" width="0.4064" layer="16"/>
 <wire x1="27.94" y1="10.16" x2="25.4" y2="7.62" width="0.4064" layer="16"/>
@@
 <wire x1="15.24" y1="5.08" x2="16.51" y2="3.81" width="0.4064" layer="1"/>
 <wire x1="16.51" y1="3.81" x2="22.86" y2="3.81" width="0.4064" layer="1"/>
-<wire x1="36.83" y1="24.13" x2="35.56" y2="24.13" width="0.4064" layer="16"/>
-<wire x1="35.56" y1="24.13" x2="33.02" y2="21.59" width="0.4064" layer="16"/>
-<wire x1="33.02" y1="21.59" x2="30.48" y2="21.59" width="0.4064" layer="16"/>
-<wire x1="30.48" y1="21.59" x2="29.21" y2="20.32" width="0.4064" layer="16"/>
-<wire x1="29.21" y1="20.32" x2="29.21" y2="19.05" width="0.4064" layer="16"/>
-<wire x1="29.21" y1="19.05" x2="27.94" y2="19.05" width="0.4064" layer="16"/>
+<contactref element="JP2" pad="4"/>
+<wire x1="27.94" y1="19.37" x2="28.26" y2="19.37" width="0.4064" layer="16"/>
+<wire x1="28.26" y1="19.37" x2="30.48" y2="21.59" width="0.4064" layer="16"/>
+<wire x1="30.48" y1="21.59" x2="33.02" y2="21.59" width="0.4064" layer="16"/>
+<wire x1="33.02" y1="21.59" x2="34.29" y2="22.86" width="0.4064" layer="16"/>
+<wire x1="34.29" y1="22.86" x2="34.29" y2="25.4" width="0.4064" layer="16"/>
+<wire x1="34.29" y1="25.4" x2="35.56" y2="26.67" width="0.4064" layer="16"/>
+<wire x1="35.56" y1="26.67" x2="36.83" y2="26.67" width="0.4064" layer="16"/>
 </signal>
 <signal name="SCL">
@@
 <contactref element="R1" pad="1"/>
 <contactref element="SV2" pad="3"/>
-<contactref element="JP2" pad="1"/>
 <wire x1="20.32" y1="5.08" x2="20.32" y2="6.35" width="0.4064" layer="1"/>
 <wire x1="20.32" y1="6.35" x2="24.13" y2="10.16" width="0.4064" layer="1"/>
@@
 <wire x1="5.08" y1="7.62" x2="21.59" y2="7.62" width="0.4064" layer="16"/>
 <wire x1="21.59" y1="7.62" x2="24.13" y2="10.16" width="0.4064" layer="16"/>
-<wire x1="24.13" y1="10.16" x2="25.4" y2="10.16" width="0.4064" layer="1"/>
-<wire x1="25.4" y1="10.16" x2="29.21" y2="13.97" width="0.4064" layer="1"/>
-<via x="29.21" y="13.97" extent="1-16" drill="0.7" shape="square"/>
-<wire x1="29.21" y1="13.97" x2="29.21" y2="17.78" width="0.4064" layer="16"/>
+<contactref element="JP2" pad="2"/>
+<wire x1="24.13" y1="10.16" x2="29.21" y2="15.24" width="0.4064" layer="1"/>
+<via x="29.21" y="15.24" extent="1-16" drill="0.7" shape="square"/>
+<wire x1="29.21" y1="15.24" x2="29.21" y2="17.78" width="0.4064" layer="16"/>
 <wire x1="29.21" y1="17.78" x2="30.48" y2="19.05" width="0.4064" layer="16"/>
-<wire x1="30.48" y1="19.05" x2="36.83" y2="19.05" width="0.4064" layer="16"/>
+<wire x1="30.48" y1="19.05" x2="33.02" y2="19.05" width="0.4064" layer="16"/>
+<wire x1="33.02" y1="19.05" x2="35.56" y2="21.59" width="0.4064" layer="16"/>
+<wire x1="35.56" y1="21.59" x2="36.83" y2="21.59" width="0.4064" layer="16"/>
 </signal>
 <signal name="SDA">
@@
 <contactref element="R2" pad="1"/>
 <contactref element="SV2" pad="1"/>
-<contactref element="JP2" pad="4"/>
 <wire x1="20.32" y1="8.89" x2="20.32" y2="10.16" width="0.4064" layer="1"/>
 <wire x1="20.32" y1="10.16" x2="22.86" y2="12.7" width="0.4064" layer="1"/>
@@
 <wire x1="7.62" y1="12.7" x2="10.16" y2="10.16" width="0.4064" layer="1"/>
 <wire x1="10.16" y1="10.16" x2="20.32" y2="10.16" width="0.4064" layer="1"/>
-<wire x1="24.13" y1="12.7" x2="25.4" y2="12.7" width="0.4064" layer="1"/>
-<wire x1="25.4" y1="12.7" x2="29.21" y2="16.51" width="0.4064" layer="1"/>
-<wire x1="29.21" y1="16.51" x2="29.21" y2="17.78" width="0.4064" layer="1"/>
-<wire x1="29.21" y1="17.78" x2="30.48" y2="19.05" width="0.4064" layer="1"/>
+<contactref element="JP2" pad="3"/>
+<wire x1="24.13" y1="12.7" x2="30.48" y2="19.05" width="0.4064" layer="1"/>
 <wire x1="30.48" y1="19.05" x2="33.02" y2="19.05" width="0.4064" layer="1"/>
 <wire x1="33.02" y1="19.05" x2="34.29" y2="20.32" width="0.4064" layer="1"/>
-<wire x1="34.29" y1="20.32" x2="34.29" y2="25.4" width="0.4064" layer="1"/>
-<wire x1="34.29" y1="25.4" x2="35.56" y2="26.67" width="0.4064" layer="1"/>
-<wire x1="35.56" y1="26.67" x2="36.83" y2="26.67" width="0.4064" layer="1"/>
+<wire x1="34.29" y1="20.32" x2="34.29" y2="22.86" width="0.4064" layer="1"/>
+<wire x1="34.29" y1="22.86" x2="35.56" y2="24.13" width="0.4064" layer="1"/>
+<wire x1="35.56" y1="24.13" x2="36.83" y2="24.13" width="0.4064" layer="1"/>
 </signal>
 <signal name="N$4">

Commit message: more layouting
Parts:
- moved R15 12.1 mm to (15.9, 2.54)
- moved IC1 4.45 mm to (27.9, 14.6)
- moved D1 3.24 mm to (15.9, 24.8)
- moved R10 2.62 mm to (15.9, 21.6)
- moved R9 2.01 mm to (15.9, 18.4)
- moved R11 1.42 mm to (15.9, 15.2)
- moved C5 1.27 mm to (36.8, 3.81)
- moved C4 1.27 mm to (36.8, 14.0)
- moved Q1 1.27 mm to (36.8, 8.89)
- moved D2 0.90 mm to (15.9, 12.1)
- moved R1 0.90 mm to (15.9, 5.71)
- moved R2 0.63 mm to (15.9, 8.89)
- moved C6 0.63 mm to (27.9, 21.0)
Connections:
- net N$27 renamed AVRD+
- net N$41 renamed AVRD-
Routing:
- net N$1: track 35.7 -> 31.9 mm
- net N$4: track 21.9 -> 18.6 mm
- net SDA: track 43.1 -> 46.2 mm
- net N$38: track 11.3 -> 8.59 mm
- net N$37: track 9.77 -> 7.64 mm
- net SCL: track 47.5 -> 46.1 mm, vias 1 -> 0
- net VCC: track 79.6 -> 78.3 mm
- net AVRD+: track 13.0 -> 12.1 mm
- net AVRD-: track 12.0 -> 12.6 mm
Other:
- board size 41.6 x 34.3 mm -> 41.6 x 29.2 mm
- board text added: "rev 1.1"
- board text removed: "rev 1"

Commit message: circuit: proper schematic
Parts:
- removed C4, C5: 22p, rcl:C0805
- removed R15: 10k, rcl:0207/10
- added C2, C3: 22p, rcl:C0805
- added R3: 1k5, rcl:0207/10
- R1: value 1k5 -> 10k
- moved D1 12.7 mm to (15.9, 12.1)
- moved D2 12.7 mm to (15.9, 24.8)
- moved R2 3.18 mm to (15.9, 5.71)
- moved R1 3.17 mm to (15.9, 2.54)
- renumbered C6 to C1, R10 to R6, R11 to R4, R9 to R5
Connections:
- net N$4 renamed MOSI
- removed net N$1: IC1.1, R15.1, SV2.5
- removed net SCL: IC1.19, JP2.2, R1.1, SV2.3
- removed net SDA: IC1.18, JP2.3, R2.1, SV2.1
- removed net VCC: C1.2, IC1.20, JP1.4, JP2.4, R1.2, R15.2, R2.2, R5.2, SV2.2
- new net +5V: C1.2, IC1.20, JP1.4, JP2.4, R1.2, R2.2, R3.2, R5.2, SV2.2
- new net MISO/SDA: IC1.18, JP2.3, R3.1, SV2.1
- new net RST: IC1.1, R1.1, SV2.5
- new net SCK/SCL: IC1.19, JP2.2, R2.1, SV2.3
- net D+: now also D1.C; no longer D2.C
- net D-: now also D2.C; no longer D1.C
- net GND: now also C2.1, C3.1; no longer C4.1, C5.1
- net N$37: now also C3.2; no longer C4.2
- net N$38: now also C2.2; no longer C5.2
Routing:
- net VCC: track 78.3 -> 0.00 mm
- net +5V: track 0.00 -> 78.3 mm
- net SDA: track 46.2 -> 0.00 mm
- net SCL: track 46.1 -> 0.00 mm
- net SCK/SCL: track 0.00 -> 46.1 mm
- net MISO/SDA: track 0.00 -> 46.1 mm
- net RST: track 0.00 -> 32.6 mm
- net N$1: track 31.9 -> 0.00 mm
- net MOSI: track 18.6 -> 38.5 mm
- net N$38: track 8.59 -> 6.87 mm
- net AVRD-: track 12.6 -> 12.1 mm

Commit message: circuit: Also, design rules...
Parts:
- moved JP2 1.91 mm to (38.7, 22.9)
Routing:
- net +5V: track 78.3 -> 80.2 mm
- net SCK/SCL: track 46.1 -> 47.6 mm
- net MISO/SDA: track 46.1 -> 47.6 mm
Changed lines of the file:
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@@
 <text x="5.715" y="23.495" size="1.016" layer="25">D-</text>
 <text x="5.715" y="20.955" size="1.016" layer="25">D+</text>
-<text x="38.735" y="23.495" size="1.016" layer="25">SDA</text>
-<text x="38.735" y="20.955" size="1.016" layer="25">SCL</text>
-<text x="38.735" y="26.035" size="1.016" layer="25">5V</text>
-<text x="38.735" y="18.415" size="1.016" layer="25">GND</text>
+<text x="34.29" y="23.495" size="1.016" layer="25">SDA</text>
+<text x="34.29" y="20.955" size="1.016" layer="25">SCL</text>
+<text x="34.925" y="26.035" size="1.016" layer="25">5V</text>
+<text x="34.29" y="18.415" size="1.016" layer="25">GND</text>
 </plain>
 <attributes>
@@
 <attribute name="VALUE" x="10.16" y="8.255" size="1.778" layer="27" ratio="10" rot="R270"/>
 </element>
-<element name="JP2" library="pinhead" package="1X04" value="I2C" x="36.83" y="22.86" smashed="yes" rot="MR90">
-<attribute name="NAME" x="38.6588" y="17.7038" size="1.27" layer="27" ratio="10" rot="MR90"/>
-<attribute name="VALUE" x="33.655" y="17.78" size="1.27" layer="28" rot="MR90"/>
+<element name="JP2" library="pinhead" package="1X04" value="I2C" x="38.735" y="22.86" smashed="yes" rot="MR90">
+<attribute name="NAME" x="40.5638" y="17.7038" size="1.27" layer="27" ratio="10" rot="MR90"/>
+<attribute name="VALUE" x="35.56" y="17.78" size="1.27" layer="28" rot="MR90"/>
 </element>
 </elements>
@@
 <wire x1="22.225" y1="19.685" x2="27.62" y2="19.685" width="0.4064" layer="16"/>
 <wire x1="27.62" y1="19.685" x2="27.94" y2="20.005" width="0.4064" layer="16"/>
-<wire x1="36.83" y1="26.67" x2="35.56" y2="26.67" width="0.4064" layer="16"/>
-<wire x1="35.56" y1="26.67" x2="33.655" y2="24.765" width="0.4064" layer="16"/>
-<wire x1="33.655" y1="24.765" x2="30.48" y2="24.765" width="0.4064" layer="16"/>
-<wire x1="30.48" y1="24.765" x2="29.845" y2="24.13" width="0.4064" layer="16"/>
-<wire x1="29.845" y1="24.13" x2="29.845" y2="20.955" width="0.4064" layer="16"/>
-<wire x1="29.845" y1="20.955" x2="29.21" y2="20.32" width="0.4064" layer="16"/>
-<wire x1="29.21" y1="20.32" x2="28.255" y2="20.32" width="0.4064" layer="16"/>
-<wire x1="28.255" y1="20.32" x2="27.94" y2="20.005" width="0.4064" layer="16"/>
 <wire x1="20.955" y1="18.415" x2="11.43" y2="8.89" width="0.4064" layer="16"/>
 <wire x1="11.43" y1="8.89" x2="10.795" y2="8.89" width="0.4064" layer="16"/>
@@
 <wire x1="21.59" y1="3.81" x2="12.065" y2="3.81" width="0.4064" layer="16"/>
 <wire x1="12.065" y1="3.81" x2="10.795" y2="2.54" width="0.4064" layer="16"/>
+<wire x1="27.94" y1="20.005" x2="28.895" y2="20.005" width="0.4064" layer="16"/>
+<wire x1="28.895" y1="20.005" x2="29.845" y2="20.955" width="0.4064" layer="16"/>
+<wire x1="29.845" y1="20.955" x2="29.845" y2="21.59" width="0.4064" layer="16"/>
+<wire x1="29.845" y1="21.59" x2="30.48" y2="22.225" width="0.4064" layer="16"/>
+<wire x1="30.48" y1="22.225" x2="33.02" y2="22.225" width="0.4064" layer="16"/>
+<wire x1="33.02" y1="22.225" x2="33.655" y2="22.86" width="0.4064" layer="16"/>
+<wire x1="33.655" y1="22.86" x2="33.655" y2="25.4" width="0.4064" layer="16"/>
+<wire x1="33.655" y1="25.4" x2="34.925" y2="26.67" width="0.4064" layer="16"/>
+<wire x1="34.925" y1="26.67" x2="38.735" y2="26.67" width="0.4064" layer="16"/>
 </signal>
 <signal name="SCK/SCL">
@@
 <wire x1="5.08" y1="7.62" x2="3.81" y2="8.89" width="0.4064" layer="1"/>
 <wire x1="20.955" y1="5.715" x2="24.13" y2="5.715" width="0.4064" layer="1"/>
-<wire x1="24.13" y1="5.715" x2="30.48" y2="12.065" width="0.4064" layer="1"/>
+<wire x1="24.13" y1="5.715" x2="24.765" y2="5.715" width="0.4064" layer="1"/>
+<wire x1="24.765" y1="5.715" x2="29.845" y2="10.795" width="0.4064" layer="1"/>
+<wire x1="29.845" y1="10.795" x2="29.845" y2="11.43" width="0.4064" layer="1"/>
+<wire x1="29.845" y1="11.43" x2="30.48" y2="12.065" width="0.4064" layer="1"/>
 <wire x1="30.48" y1="12.065" x2="33.02" y2="12.065" width="0.4064" layer="1"/>
 <wire x1="33.02" y1="12.065" x2="34.925" y2="13.97" width="0.4064" layer="1"/>
-<wire x1="34.925" y1="13.97" x2="34.925" y2="20.955" width="0.4064" layer="1"/>
-<wire x1="34.925" y1="20.955" x2="35.56" y2="21.59" width="0.4064" layer="1"/>
-<wire x1="35.56" y1="21.59" x2="36.83" y2="21.59" width="0.4064" layer="1"/>
+<wire x1="34.925" y1="13.97" x2="34.925" y2="19.685" width="0.4064" layer="1"/>
+<wire x1="34.925" y1="19.685" x2="36.83" y2="21.59" width="0.4064" layer="1"/>
+<wire x1="36.83" y1="21.59" x2="38.735" y2="21.59" width="0.4064" layer="1"/>
 </signal>
 <signal name="MISO/SDA">
@@
 <wire x1="22.225" y1="8.89" x2="22.86" y2="8.255" width="0.4064" layer="1"/>
 <wire x1="22.86" y1="8.255" x2="24.13" y2="8.255" width="0.4064" layer="1"/>
-<wire x1="24.13" y1="8.255" x2="30.48" y2="14.605" width="0.4064" layer="1"/>
+<wire x1="24.13" y1="8.255" x2="24.765" y2="8.255" width="0.4064" layer="1"/>
+<wire x1="24.765" y1="8.255" x2="29.845" y2="13.335" width="0.4064" layer="1"/>
+<wire x1="29.845" y1="13.335" x2="29.845" y2="13.97" width="0.4064" layer="1"/>
+<wire x1="29.845" y1="13.97" x2="30.48" y2="14.605" width="0.4064" layer="1"/>
 <wire x1="30.48" y1="14.605" x2="33.02" y2="14.605" width="0.4064" layer="1"/>
 <wire x1="33.02" y1="14.605" x2="33.655" y2="15.24" width="0.4064" layer="1"/>
-<wire x1="33.655" y1="15.24" x2="33.655" y2="22.225" width="0.4064" layer="1"/>
-<wire x1="33.655" y1="22.225" x2="35.56" y2="24.13" width="0.4064" layer="1"/>
-<wire x1="35.56" y1="24.13" x2="36.83" y2="24.13" width="0.4064" layer="1"/>
+<wire x1="33.655" y1="15.24" x2="33.655" y2="20.955" width="0.4064" layer="1"/>
+<wire x1="33.655" y1="20.955" x2="36.83" y2="24.13" width="0.4064" layer="1"/>
+<wire x1="36.83" y1="24.13" x2="38.735" y2="24.13" width="0.4064" layer="1"/>
 </signal>
 <signal name="MOSI">

Commit message: tht circuit: preparing rev 2
Parts:
- added LED1: act, led:LED3MM
- added LED2: pwr, led:LED3MM
- added R7: 150..1k, rcl:0207/10
- moved D1 13.3 mm to (15.9, 25.4)
- moved R1 7.62 mm to (15.9, 10.2)
- moved R2 6.98 mm to (15.9, 12.7)
- moved R3 6.35 mm to (15.9, 15.2)
- moved R4 2.54 mm to (15.9, 17.8)
- moved D2 2.54 mm to (15.9, 27.3)
- moved R5 1.91 mm to (15.9, 20.3)
- moved R6 1.27 mm to (15.9, 22.9)
Connections:
- new net EAE: LED1.K, LED2.A, R7.1
- new net LED1: IC1.3, R7.2
- new net LED2: IC1.2, LED1.A, LED2.K
Routing:
- net LED1: track 0.00 -> 25.6 mm
- net LED2: track 0.00 -> 19.6 mm
- net MOSI: track 38.5 -> 20.1 mm, vias 0 -> 1
- net EAE: track 0.00 -> 8.04 mm
- net SCK/SCL: track 47.6 -> 53.6 mm, vias 0 -> 1
- net MISO/SDA: track 47.6 -> 53.0 mm
- net RST: track 32.6 -> 37.1 mm, vias 0 -> 1
- net D+: track 13.3 -> 17.2 mm
- net +5V: track 80.2 -> 82.6 mm
- net AVRD-: track 12.1 -> 12.6 mm
- net AVRD+: track 12.1 -> 11.6 mm
Other:
- board text added: "ACT"
- board text added: "CC-BY"
- board text added: "PWR"
- board text added: "b"
- board text added: "by derf"
- board text added: "g"
- board text added: "r"
- board text added: "rev 2"
- board text added: "w"
- board text removed: "derf"
- board text removed: "rev 1.1"
