File: circuit/circuit.sch (EAGLE design)
At the start: 16 parts, among them IC1 AT90S2313P, Q1 16MHz

Commit message: tht circuit: preparing rev 2
Parts:
- added LED1: act, led:LED3MM
- added LED2: pwr, led:LED3MM
- added R7: 150..1k, rcl:R-EU_0207/10
Connections:
- new net EAE: LED1.C, LED2.A, R7.1
- new net LED1: IC1.(TXD)PD1, R7.2
- new net LED2: IC1.(RXD)PD0, LED1.A, LED2.C
Other:
- note added: "Status LED"
Changed lines of the file:
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@@
 <part name="GND3" library="supply1" deviceset="GND" device=""/>
 <part name="FRAME1" library="frames" deviceset="A5L-LOC" device="" value="vusb-i2c"/>
+<part name="LED1" library="led" deviceset="LED" device="3MM" value="act"/>
+<part name="LED2" library="led" deviceset="LED" device="3MM" value="pwr"/>
+<part name="R7" library="rcl" deviceset="R-EU_" device="0207/10" value="150..1k"/>
 </parts>
 <sheets>
@@
 <wire x1="85.09" y1="53.34" x2="85.09" y2="4.064" width="0.1524" layer="97" style="longdash"/>
 <wire x1="86.36" y1="53.34" x2="116.84" y2="53.34" width="0.1524" layer="97" style="longdash"/>
-<wire x1="116.84" y1="53.34" x2="116.84" y2="129.54" width="0.1524" layer="97" style="longdash"/>
+<wire x1="116.84" y1="53.34" x2="116.84" y2="104.14" width="0.1524" layer="97" style="longdash"/>
+<wire x1="116.84" y1="104.14" x2="116.84" y2="129.54" width="0.1524" layer="97" style="longdash"/>
 <wire x1="116.84" y1="53.34" x2="180.34" y2="53.34" width="0.1524" layer="97" style="longdash"/>
 <text x="63.5" y="50.8" size="1.778" layer="97">USB Interface</text>
@@
 <text x="119.38" y="55.88" size="1.778" layer="97">I2C Interface</text>
 <text x="86.36" y="50.8" size="1.778" layer="97">SPI Interface</text>
+<wire x1="116.84" y1="104.14" x2="180.34" y2="104.14" width="0.1524" layer="97" style="longdash"/>
+<text x="119.38" y="124.46" size="1.778" layer="97">Status LED</text>
 </plain>
 <instances>
@@
 <instance part="GND3" gate="1" x="157.48" y="63.5"/>
 <instance part="FRAME1" gate="G$1" x="0" y="0"/>
+<instance part="LED1" gate="G$1" x="142.24" y="121.92" rot="R90"/>
+<instance part="LED2" gate="G$1" x="144.78" y="111.76" rot="R270"/>
+<instance part="R7" gate="G$1" x="157.48" y="116.84"/>
 </instances>
 <busses>
@@
 </segment>
 </net>
+<net name="LED2" class="0">
+<segment>
+<pinref part="IC1" gate="G$1" pin="(RXD)PD0"/>
+<wire x1="76.2" y1="58.42" x2="78.74" y2="58.42" width="0.1524" layer="91"/>
+<wire x1="78.74" y1="58.42" x2="78.74" y2="55.88" width="0.1524" layer="91"/>
+<wire x1="78.74" y1="55.88" x2="101.6" y2="55.88" width="0.1524" layer="91"/>
+<label x="96.52" y="55.88" size="1.778" layer="95"/>
+</segment>
+<segment>
+<pinref part="LED2" gate="G$1" pin="C"/>
+<wire x1="137.16" y1="111.76" x2="139.7" y2="111.76" width="0.1524" layer="91"/>
+<wire x1="137.16" y1="111.76" x2="137.16" y2="116.84" width="0.1524" layer="91"/>
+<pinref part="LED1" gate="G$1" pin="A"/>
+<wire x1="137.16" y1="116.84" x2="137.16" y2="121.92" width="0.1524" layer="91"/>
+<wire x1="137.16" y1="121.92" x2="139.7" y2="121.92" width="0.1524" layer="91"/>
+<wire x1="137.16" y1="116.84" x2="121.92" y2="116.84" width="0.1524" layer="91"/>
+<junction x="137.16" y="116.84"/>
+<label x="121.92" y="116.84" size="1.778" layer="95"/>
+</segment>
+</net>
+<net name="LED1" class="0">
+<segment>
+<pinref part="IC1" gate="G$1" pin="(TXD)PD1"/>
+<wire x1="76.2" y1="60.96" x2="81.28" y2="60.96" width="0.1524" layer="91"/>
+<wire x1="81.28" y1="60.96" x2="81.28" y2="58.42" width="0.1524" layer="91"/>
+<wire x1="81.28" y1="58.42" x2="101.6" y2="58.42" width="0.1524" layer="91"/>
+<label x="96.52" y="58.42" size="1.778" layer="95"/>
+</segment>
+<segment>
+<pinref part="R7" gate="G$1" pin="2"/>
+<wire x1="162.56" y1="116.84" x2="175.26" y2="116.84" width="0.1524" layer="91"/>
+<label x="170.18" y="116.84" size="1.778" layer="95"/>
+</segment>
+</net>
+<net name="EAE" class="0">
+<segment>
+<pinref part="LED1" gate="G$1" pin="C"/>
+<wire x1="147.32" y1="121.92" x2="149.86" y2="121.92" width="0.1524" layer="91"/>
+<pinref part="LED2" gate="G$1" pin="A"/>
+<wire x1="149.86" y1="121.92" x2="149.86" y2="116.84" width="0.1524" layer="91"/>
+<wire x1="149.86" y1="116.84" x2="149.86" y2="111.76" width="0.1524" layer="91"/>
+<wire x1="149.86" y1="111.76" x2="147.32" y2="111.76" width="0.1524" layer="91"/>
+<pinref part="R7" gate="G$1" pin="1"/>
+<wire x1="152.4" y1="116.84" x2="149.86" y2="116.84" width="0.1524" layer="91"/>
+<junction x="149.86" y="116.84"/>
+</segment>
+</net>
